Commit message: Update wheelchair config

File: urdf/wheelchair_simplified.urdf (robot description, URDF)
Before this commit: robot arlobot_hardware, 5 links, 4 joints
Joints:
- joint zed_base: origin xyz=-0.385 0 -0.49 rpy=0 0 0 -> xyz=-0.33 -0.01 -0.28 rpy=0 0 0
- joint zed_footprint: origin xyz=0 0 0.49 rpy=0 0 0 -> xyz=0 0 0.28 rpy=0 0 0
